File: X16-Pi-Shield.brd (EAGLE design)
At the start: 160 x 100 mm, 51 parts, among them J1 CONN_DF13-4P-1.25DSA, J2 CONN_DF13-4P-1.25DSA, J3 CONN_DF13-4P-1.25DSA, J4 SAMTEC-HTST-110-04-X-D-RAJ, Q2 2.5A/30V/105mΩ, Q3 220mA/50V/3.5Ω, U1 INA260AIPW, U2 AZ1117IH-3.3TRG1, Y2 ECS-80-S-4X

Commit message: update
Parts:
- removed J1, J2: CONN_DF13-4P-1.25DSA, X16-Pi-Shield:DF13-4P-1.25DSA
- added J5: BM04B-GHS-TBT, X16-Pi-Shield:CONN_BM04B-GHS-TBT_JST
- moved U1 457.8 mm to (63.5, 67.3), turned to 270 degrees
- moved C5 447.4 mm to (36.8, 48.3)
- moved JP5 447.4 mm to (40.6, 38.1)
- moved JP8 447.4 mm to (40.6, 33.0)
- moved TP4 447.4 mm to (35.6, 44.5)
- moved TP5 447.4 mm to (35.6, 41.9)
- moved U$4 414.7 mm to (36.8, 25.4)
- moved U2 411.8 mm to (59.7, 20.3)
- moved C4 408.7 mm to (59.7, 7.62)
- moved U$2 408.2 mm to (35.6, 49.5)
- moved C3 387.1 mm to (45.7, 19.1)
- moved JP7 387.1 mm to (49.5, 22.9)
- moved J4 362.3 mm to (111.8, 17.8)
- moved OVERCURRENT 313.2 mm to (24.1, 35.6)
- moved Q2 313.2 mm to (24.1, 45.7)
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Connections:
- net 3V3: now also J5.2; no longer J1.1, J2.1
- net GND: now also J5.1; no longer J1.4, J2.4
- net SCL: now also J5.3; no longer J1.2, J2.2
- net SDA: now also J5.4; no longer J1.3, J2.3
Other:
- board size 160 x 100 mm -> 69.9 x 73 mm
