File: X16-Pi-Shield.brd (EAGLE design)
At the start: 81.3 x 74.3 mm, 36 parts, among them J3 CONN_DF13-4P-1.25DSA, J4 HTST-110-04-L-D-RA, J5 BM04B-GHS-TBT, U1 INA260AIPW, U2 AZ1117IH-3.3TRG1

Commit message: more traces
Routing:
- net GND: track 6.13 -> 21.7 mm, vias 6 -> 13
- net 5V_EXT: track 57.2 -> 59.6 mm
- net 5V: track 160.7 -> 161.6 mm
- net SDA: track 224.7 -> 225.4 mm
Changed lines of the file:
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@@
 <wire x1="8.2677" y1="25.31374375" x2="8.2677" y2="23.7871" width="0.2032" layer="16"/>
 <via x="33.274" y="48.514" extent="1-16" drill="0.35"/>
-<wire x1="25.867" y1="13.513" x2="25.867" y2="19.253" width="0" layer="19" extent="1-1"/>
-<wire x1="22.846" y1="24.84" x2="25.867" y2="19.253" width="0" layer="19" extent="1-1"/>
-<wire x1="33.616" y1="24.638" x2="25.867" y2="19.253" width="0" layer="19" extent="1-1"/>
-<wire x1="7.1882" y1="17.2466" x2="3.556" y2="15.533" width="0" layer="19" extent="1-1"/>
+<via x="26.924" y="17.526" extent="1-16" drill="0.35"/>
+<via x="26.797" y="12.192" extent="1-16" drill="0.35"/>
+<wire x1="25.867" y1="13.513" x2="26.0834" y2="13.2966" width="0.1524" layer="1"/>
+<wire x1="26.0834" y1="13.2966" x2="26.0834" y2="12.66333125" width="0.1524" layer="1"/>
+<wire x1="26.0834" y1="12.66333125" x2="26.24733125" y2="12.4994" width="0.1524" layer="1"/>
+<wire x1="26.24733125" y1="12.4994" x2="26.4896" y2="12.4994" width="0.1524" layer="1"/>
+<wire x1="26.4896" y1="12.4994" x2="26.797" y2="12.192" width="0.1524" layer="1"/>
+<wire x1="26.924" y1="17.526" x2="25.867" y2="18.583" width="0.1524" layer="1"/>
+<wire x1="25.867" y1="18.583" x2="25.867" y2="19.253" width="0.1524" layer="1"/>
+<via x="30.099" y="16.256" extent="1-16" drill="0.35"/>
+<via x="28.702" y="17.399" extent="1-16" drill="0.35"/>
+<wire x1="30.099" y1="16.256" x2="29.845" y2="16.256" width="0.762" layer="16"/>
+<wire x1="29.845" y1="16.256" x2="28.702" y2="17.399" width="0.762" layer="16"/>
+<via x="23.368" y="22.606" extent="1-16" drill="0.35"/>
+<via x="32.766" y="22.606" extent="1-16" drill="0.35"/>
+<wire x1="29.7214" y1="20.2156" x2="30.3756" y2="20.2156" width="0.762" layer="16"/>
+<wire x1="30.3756" y1="20.2156" x2="32.766" y2="22.606" width="0.762" layer="16"/>
+<wire x1="28.702" y1="17.399" x2="28.702" y2="19.1962" width="0.762" layer="16"/>
+<wire x1="28.702" y1="19.1962" x2="29.7214" y2="20.2156" width="0.762" layer="16"/>
+<wire x1="33.447" y1="24.469" x2="33.616" y2="24.638" width="0.762" layer="1"/>
+<wire x1="33.447" y1="23.86175625" x2="33.447" y2="24.469" width="0.762" layer="1"/>
+<wire x1="32.766" y1="22.606" x2="32.766" y2="23.18075625" width="0.762" layer="1"/>
+<wire x1="32.766" y1="23.18075625" x2="33.447" y2="23.86175625" width="0.762" layer="1"/>
+<via x="55.372" y="26.797" extent="1-16" drill="0.35"/>
+<wire x1="7.1882" y1="27.4066" x2="7.1882" y2="35.0266" width="0" layer="19" extent="1-1"/>
+<wire x1="7.1882" y1="17.2466" x2="9.7282" y2="22.3266" width="0" layer="19" extent="1-1"/>
+<wire x1="3.556" y1="15.533" x2="7.1882" y2="17.2466" width="0" layer="19" extent="1-1"/>
 <wire x1="7.1882" y1="47.7266" x2="7.1882" y2="52.8066" width="0" layer="19" extent="1-1"/>
 <wire x1="12.573" y1="15.787" x2="7.1882" y2="17.2466" width="0" layer="19" extent="1-1"/>
-<wire x1="9.7282" y1="22.3266" x2="7.1882" y2="17.2466" width="0" layer="19" extent="1-1"/>
 <wire x1="9.7282" y1="42.6466" x2="7.1882" y2="47.7266" width="0" layer="19" extent="1-1"/>
-<wire x1="7.1882" y1="35.0266" x2="7.1882" y2="27.4066" width="0" layer="19" extent="1-1"/>
 <wire x1="-6.35" y1="27.559" x2="7.1882" y2="27.4066" width="0" layer="19" extent="1-1"/>
 </signal>
@@
 <wire x1="-9.3952" y1="43.18786875" x2="-9.3952" y2="13.92735625" width="0.2032" layer="16"/>
 <wire x1="-9.3952" y1="13.92735625" x2="-6.26284375" y2="10.795" width="0.2032" layer="16"/>
-<wire x1="27.167" y1="13.513" x2="27.178" y2="13.502" width="0.2032" layer="1"/>
-<wire x1="27.178" y1="13.502" x2="27.178" y2="12.192" width="0.2032" layer="1"/>
-<via x="27.178" y="12.192" extent="1-16" drill="0.35"/>
-<wire x1="27.178" y1="12.192" x2="26.035" y2="11.049" width="0.2032" layer="16"/>
+<wire x1="27.167" y1="13.513" x2="27.813" y2="12.867" width="0.2032" layer="1"/>
+<wire x1="27.813" y1="12.867" x2="27.813" y2="12.192" width="0.2032" layer="1"/>
+<via x="27.813" y="12.192" extent="1-16" drill="0.35"/>
+<wire x1="27.813" y1="12.192" x2="26.67" y2="11.049" width="0.2032" layer="16"/>
 <wire x1="13.3858" y1="11.049" x2="9.7282" y2="14.7066" width="0.2032" layer="16"/>
-<wire x1="26.035" y1="11.049" x2="13.3858" y2="11.049" width="0.2032" layer="16"/>
+<wire x1="26.67" y1="11.049" x2="13.3858" y2="11.049" width="0.2032" layer="16"/>
 <wire x1="63.871" y1="18.542" x2="62.611" y2="19.802" width="0.2032" layer="1"/>
 <wire x1="62.611" y1="19.802" x2="62.611" y2="21.844" width="0.2032" layer="1"/>
@@
 <wire x1="57.531" y1="24.765" x2="57.531" y2="28.956" width="0.2032" layer="1"/>
 <wire x1="57.531" y1="28.956" x2="57.277" y2="29.21" width="0.2032" layer="1"/>
-<wire x1="27.167" y1="13.513" x2="27.762" y2="13.513" width="0.2032" layer="1"/>
-<wire x1="27.762" y1="13.513" x2="28.448" y2="12.827" width="0.2032" layer="1"/>
-<via x="28.448" y="12.827" extent="1-16" drill="0.35"/>
-<wire x1="28.448" y1="12.827" x2="40.386" y2="24.765" width="0.2032" layer="16"/>
+<wire x1="27.167" y1="13.513" x2="28.016" y2="13.513" width="0.2032" layer="1"/>
+<wire x1="28.016" y1="13.513" x2="28.575" y2="12.954" width="0.2032" layer="1"/>
+<via x="28.575" y="12.954" extent="1-16" drill="0.35"/>
+<wire x1="28.575" y1="12.954" x2="40.386" y2="24.765" width="0.2032" layer="16"/>
 <wire x1="40.386" y1="24.765" x2="57.531" y2="24.765" width="0.2032" layer="16"/>
 <wire x1="57.277" y1="29.21" x2="57.277" y2="35.052" width="0.2032" layer="1"/>
@@
 <wire x1="18.242" y1="16.683" x2="18.288" y2="16.637" width="0.2032" layer="1"/>
 <wire x1="11.9677875" y1="16.683" x2="18.242" y2="16.683" width="0.2032" layer="1"/>
-<via x="28.829" y="16.129" extent="1-16" drill="0.35"/>
+<via x="28.448" y="16.002" extent="1-16" drill="0.35"/>
 <wire x1="24.75713125" y1="14.2268" x2="25.28086875" y2="14.2268" width="0.2032" layer="16"/>
 <wire x1="18.288" y1="16.637" x2="22.34693125" y2="16.637" width="0.2032" layer="16"/>
 <wire x1="22.34693125" y1="16.637" x2="24.75713125" y2="14.2268" width="0.2032" layer="16"/>
-<wire x1="27.18306875" y1="16.129" x2="28.829" y2="16.129" width="0.2032" layer="16"/>
-<wire x1="25.28086875" y1="14.2268" x2="27.18306875" y2="16.129" width="0.2032" layer="16"/>
-<wire x1="28.829" y1="16.129" x2="30.099" y2="17.399" width="0.2032" layer="1"/>
+<wire x1="27.05606875" y1="16.002" x2="28.448" y2="16.002" width="0.2032" layer="16"/>
+<wire x1="25.28086875" y1="14.2268" x2="27.05606875" y2="16.002" width="0.2032" layer="16"/>
+<wire x1="29.845" y1="17.399" x2="30.099" y2="17.399" width="0.2032" layer="1"/>
+<wire x1="29.845" y1="17.399" x2="28.448" y2="16.002" width="0.2032" layer="1"/>
 <via x="30.099" y="17.399" extent="1-16" drill="0.35"/>
 <wire x1="30.099" y1="17.399" x2="30.099" y2="19.304" width="0.2032" layer="16"/>
@@
 <wire x1="-2.921" y1="66.802" x2="-1.397" y2="65.278" width="0.762" layer="1"/>
 <wire x1="-1.397" y1="65.278" x2="-1.397" y2="57.873" width="0.762" layer="1"/>
-<via x="9.144" y="0.889" extent="1-16" drill="0.35"/>
+<via x="7.62" y="-0.127" extent="1-16" drill="0.35"/>
 <wire x1="-0.67605625" y1="57.2564" x2="-0.3636" y2="56.94394375" width="0.762" layer="1"/>
-<wire x1="9.0678" y1="0.9652" x2="9.144" y2="0.889" width="0.762" layer="1"/>
 <wire x1="-1.397" y1="57.873" x2="-0.7804" y2="57.2564" width="0.762" layer="1"/>
 <wire x1="-0.7804" y1="57.2564" x2="-0.67605625" y2="57.2564" width="0.762" layer="1"/>
@@
 <wire x1="-0.3636" y1="53.74743125" x2="-7.6454" y2="46.46563125" width="0.762" layer="1"/>
 <wire x1="-7.6454" y1="46.46563125" x2="-7.6454" y2="6.702425" width="0.762" layer="1"/>
-<wire x1="-7.6454" y1="6.702425" x2="-1.908175" y2="0.9652" width="0.762" layer="1"/>
-<wire x1="-1.908175" y1="0.9652" x2="9.0678" y2="0.9652" width="0.762" layer="1"/>
-<wire x1="9.144" y1="0.889" x2="11.303" y2="3.048" width="0.762" layer="16"/>
+<wire x1="-7.6454" y1="6.702425" x2="-0.765175" y2="-0.1778" width="0.762" layer="1"/>
+<wire x1="7.62" y1="-0.127" x2="7.5692" y2="-0.1778" width="0.762" layer="1"/>
+<wire x1="7.5692" y1="-0.1778" x2="-0.765175" y2="-0.1778" width="0.762" layer="1"/>
+<wire x1="7.62" y1="-0.127" x2="10.795" y2="3.048" width="0.762" layer="16"/>
 <via x="12.446" y="3.048" extent="1-16" drill="0.35"/>
 <wire x1="12.446" y1="3.048" x2="15.3924" y2="3.048" width="0.762" layer="1"/>
 <wire x1="15.3924" y1="3.048" x2="15.50781875" y2="2.93258125" width="0.762" layer="1"/>
-<wire x1="11.303" y1="3.048" x2="12.446" y2="3.048" width="0.762" layer="16"/>
+<wire x1="10.795" y1="3.048" x2="12.446" y2="3.048" width="0.762" layer="16"/>
 <wire x1="22.617" y1="19.253" x2="15.748" y2="12.384" width="0.762" layer="1"/>
 <wire x1="15.748" y1="12.384" x2="15.748" y2="3.1727625" width="0.762" layer="1"/>
@@
 <contactref element="JP9" pad="2"/>
 <contactref element="J4" pad="20"/>
-<wire x1="15.748" y1="1.8796" x2="-0.9906" y2="1.8796" width="0.762" layer="1"/>
-<wire x1="-0.9906" y1="1.8796" x2="-6.35" y2="7.239" width="0.762" layer="1"/>
-<wire x1="15.748" y1="1.8796" x2="22.617" y2="8.7486" width="0.762" layer="1"/>
-<wire x1="22.617" y1="8.7486" x2="22.617" y2="13.513" width="0.762" layer="1"/>
+<wire x1="15.748" y1="1.8796" x2="15.748" y2="0.9906" width="0.762" layer="1"/>
+<wire x1="15.748" y1="0.9906" x2="-0.1016" y2="0.9906" width="0.762" layer="1"/>
+<wire x1="-0.1016" y1="0.9906" x2="-6.35" y2="7.239" width="0.762" layer="1"/>
+<wire x1="22.617" y1="6.8436" x2="17.653" y2="1.8796" width="0.762" layer="1"/>
+<wire x1="15.748" y1="1.8796" x2="17.653" y2="1.8796" width="0.762" layer="1"/>
+<wire x1="22.617" y1="6.8436" x2="22.617" y2="13.513" width="0.762" layer="1"/>
 <wire x1="22.617" y1="13.513" x2="23.267" y2="13.513" width="0.762" layer="1"/>
 <wire x1="23.267" y1="13.513" x2="23.8286" y2="13.513" width="0.762" layer="1"/>

Commit message: more
Routing:
- net 3V3: track 163.6 -> 247.4 mm, vias 0 -> 6
- net SCL: track 208.4 -> 217.7 mm, vias 7 -> 8
Changed lines of the file:
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@@
 <wire x1="50.419" y1="52.324" x2="50.419" y2="56.222" width="0.762" layer="1"/>
 <wire x1="50.419" y1="56.222" x2="50.458" y2="56.261" width="0.762" layer="1"/>
+<wire x1="-9.271" y1="52.285" x2="-7.454" y2="52.285" width="0.762" layer="1"/>
+<wire x1="-7.454" y1="52.285" x2="-5.207" y2="50.038" width="0.762" layer="1"/>
+<via x="-5.207" y="50.038" extent="1-16" drill="0.35"/>
+<wire x1="-5.207" y1="50.038" x2="-5.207" y2="42.037" width="0.762" layer="16"/>
+<wire x1="-5.207" y1="42.037" x2="-5.588" y2="41.656" width="0.762" layer="16"/>
+<via x="-5.588" y="41.656" extent="1-16" drill="0.35"/>
+<wire x1="-5.588" y1="41.656" x2="-5.588" y2="33.02" width="0.762" layer="1"/>
+<wire x1="-5.588" y1="33.02" x2="-5.715" y2="32.893" width="0.762" layer="1"/>
+<via x="-5.715" y="32.893" extent="1-16" drill="0.35"/>
+<wire x1="-5.715" y1="32.893" x2="-6.096" y2="32.512" width="0.762" layer="16"/>
+<via x="-8.763" y="32.512" extent="1-16" drill="0.35"/>
+<wire x1="-6.096" y1="32.512" x2="-8.7602" y2="32.512" width="0.762" layer="16"/>
+<wire x1="-8.7602" y1="32.512" x2="-8.7602" y2="14.478" width="0.762" layer="16"/>
+<via x="-8.7602" y="14.478" extent="1-16" drill="0.35"/>
+<wire x1="-8.7602" y1="14.478" x2="-8.7602" y2="4.4422" width="0.762" layer="1"/>
+<wire x1="-8.7602" y1="4.4422" x2="-7.62" y2="3.302" width="0.762" layer="1"/>
+<via x="-7.62" y="3.302" extent="1-16" drill="0.35"/>
+<wire x1="-7.62" y1="3.302" x2="-0.432425" y2="3.302" width="0.762" layer="16"/>
+<wire x1="-0.432425" y1="3.302" x2="0.532775" y2="4.2672" width="0.762" layer="16"/>
+<wire x1="0.532775" y1="4.2672" x2="3.2512" y2="4.2672" width="0.762" layer="16"/>
+<wire x1="5.688" y1="6.704" x2="5.688" y2="8.4582" width="0.762" layer="16"/>
+<wire x1="5.688" y1="8.4582" x2="7.3118" y2="10.082" width="0.762" layer="16"/>
+<wire x1="7.3118" y1="10.082" x2="7.632" y2="10.082" width="0.762" layer="16"/>
+<wire x1="7.632" y1="10.082" x2="9.73" y2="12.18" width="0.762" layer="16"/>
+<wire x1="3.2512" y1="4.2672" x2="5.688" y2="6.704" width="0.762" layer="16"/>
+<wire x1="11.5396" y1="16.55794375" x2="11.85205625" y2="16.8704" width="0.762" layer="1"/>
+<wire x1="9.73" y1="12.18" x2="11.5396" y2="13.9896" width="0.762" layer="1"/>
+<wire x1="11.85205625" y1="16.8704" x2="11.9564" y2="16.8704" width="0.762" layer="1"/>
+<wire x1="11.9564" y1="16.8704" x2="12.573" y2="17.487" width="0.762" layer="1"/>
+<wire x1="11.5396" y1="13.9896" x2="11.5396" y2="16.55794375" width="0.762" layer="1"/>
 <wire x1="40.767" y1="59.5884" x2="40.767" y2="59.6265" width="0" layer="19" extent="1-1"/>
-<wire x1="9.73" y1="12.18" x2="12.573" y2="17.487" width="0" layer="19" extent="1-1"/>
-<wire x1="-9.271" y1="48.475" x2="9.7282" y2="32.4866" width="0" layer="19" extent="1-1"/>
+<wire x1="-8.763" y1="32.512" x2="-5.715" y2="32.893" width="0" layer="19" extent="1-1"/>
 </signal>
 <signal name="SCL">
@@
 <wire x1="58.6232" y1="46.49550625" x2="58.6232" y2="51.7398" width="0.2032" layer="1"/>
 <via x="18.288" y="16.637" extent="1-16" drill="0.35"/>
-<wire x1="9.7282" y1="17.2466" x2="11.4041875" y2="17.2466" width="0.2032" layer="1"/>
-<wire x1="11.4041875" y1="17.2466" x2="11.9677875" y2="16.683" width="0.2032" layer="1"/>
-<wire x1="18.242" y1="16.683" x2="18.288" y2="16.637" width="0.2032" layer="1"/>
-<wire x1="11.9677875" y1="16.683" x2="18.242" y2="16.683" width="0.2032" layer="1"/>
 <via x="28.448" y="16.002" extent="1-16" drill="0.35"/>
 <wire x1="24.75713125" y1="14.2268" x2="25.28086875" y2="14.2268" width="0.2032" layer="16"/>
-<wire x1="18.288" y1="16.637" x2="22.34693125" y2="16.637" width="0.2032" layer="16"/>
+<wire x1="18.288" y1="16.637" x2="18.415" y2="16.637" width="0.2032" layer="16"/>
+<wire x1="18.415" y1="16.637" x2="22.34693125" y2="16.637" width="0.2032" layer="16"/>
 <wire x1="22.34693125" y1="16.637" x2="24.75713125" y2="14.2268" width="0.2032" layer="16"/>
 <wire x1="27.05606875" y1="16.002" x2="28.448" y2="16.002" width="0.2032" layer="16"/>
@@
 <wire x1="37.211" y1="54.102" x2="35.804" y2="52.695" width="0.2032" layer="1"/>
 <wire x1="35.804" y1="52.695" x2="35.804" y2="51.1255" width="0.2032" layer="1"/>
+<wire x1="9.7282" y1="17.2466" x2="11.6614" y2="19.1798" width="0.2032" layer="1"/>
+<wire x1="11.6614" y1="19.1798" x2="11.6614" y2="21.28746875" width="0.2032" layer="1"/>
+<via x="11.6614" y="21.28746875" extent="1-16" drill="0.35"/>
+<wire x1="11.6614" y1="21.28746875" x2="14.50393125" y2="24.13" width="0.2032" layer="16"/>
+<wire x1="14.50393125" y1="24.13" x2="14.732" y2="24.13" width="0.2032" layer="16"/>
+<wire x1="14.732" y1="24.13" x2="18.415" y2="20.447" width="0.2032" layer="16"/>
+<wire x1="18.415" y1="20.447" x2="18.415" y2="16.637" width="0.2032" layer="16"/>
 </signal>
 <signal name="5V">
@@
 <wire x1="-1.397" y1="57.873" x2="-0.7804" y2="57.2564" width="0.762" layer="1"/>
 <wire x1="-0.7804" y1="57.2564" x2="-0.67605625" y2="57.2564" width="0.762" layer="1"/>
-<wire x1="-0.3636" y1="56.94394375" x2="-0.3636" y2="53.74743125" width="0.762" layer="1"/>
-<wire x1="-0.3636" y1="53.74743125" x2="-7.6454" y2="46.46563125" width="0.762" layer="1"/>
-<wire x1="-7.6454" y1="46.46563125" x2="-7.6454" y2="6.702425" width="0.762" layer="1"/>
+<wire x1="-0.3636" y1="56.94394375" x2="-0.3636" y2="52.85843125" width="0.762" layer="1"/>
+<wire x1="-0.3636" y1="52.85843125" x2="-7.6454" y2="45.57663125" width="0.762" layer="1"/>
+<wire x1="-7.6454" y1="45.57663125" x2="-7.6454" y2="6.702425" width="0.762" layer="1"/>
 <wire x1="-7.6454" y1="6.702425" x2="-0.765175" y2="-0.1778" width="0.762" layer="1"/>
 <wire x1="7.62" y1="-0.127" x2="7.5692" y2="-0.1778" width="0.762" layer="1"/>
@@
 <contactref element="TP4" pad="1"/>
 <contactref element="J4" pad="2"/>
-<wire x1="-6.35" y1="30.099" x2="-6.35" y2="46.863" width="0.2032" layer="1"/>
-<wire x1="7.1882" y1="60.4266" x2="7.1882" y2="60.4012" width="0.2032" layer="1"/>
-<wire x1="7.1882" y1="60.4012" x2="-6.35" y2="46.863" width="0.2032" layer="1"/>
+<wire x1="-4.318" y1="48.006" x2="-4.318" y2="32.131" width="0.2032" layer="1"/>
+<wire x1="-6.35" y1="30.099" x2="-4.318" y2="32.131" width="0.2032" layer="1"/>
+<wire x1="7.1882" y1="60.4266" x2="7.1882" y2="59.5122" width="0.2032" layer="1"/>
+<wire x1="7.1882" y1="59.5122" x2="-4.318" y2="48.006" width="0.2032" layer="1"/>
 <wire x1="7.1882" y1="60.4266" x2="3.556" y2="64.0588" width="0.2032" layer="1"/>
 <wire x1="3.556" y1="64.0588" x2="3.556" y2="66.802" width="0.2032" layer="1"/>

Commit message: stuff
Parts:
- moved C8 0.36 mm to (12.3, 16.9), turned to 180 degrees
Routing:
- net GND: track 21.7 -> 50.8 mm, vias 13 -> 17
- net SCL: track 217.7 -> 213.0 mm
- net 5V_EXT: track 59.6 -> 58.2 mm
- net 5V: track 161.6 -> 162.4 mm

Commit message: remade the board
Parts:
- moved J9 74.4 mm to (74.9, 12.7), turned to 270 degrees
- moved R12 71.8 mm to (61.7, 58.2), turned to 0 degrees
- moved R11 70.9 mm to (61.6, 54.6), turned to 0 degrees
- moved TP7 66.8 mm to (16.6, 2.92)
- moved C8 65.4 mm to (61.7, 59.7)
- moved J12 65.3 mm to (42.4, 2.54), turned to 0 degrees
- moved J15 60.4 mm to (74.9, 19.1), turned to 90 degrees
- moved 5V 58.4 mm to (18.9, 3.56), turned to 0 degrees
- moved JP5 58.1 mm to (3.30, 4.57), turned to 270 degrees
- moved R15 56.0 mm to (20.2, 5.33), turned to 0 degrees
- moved J14 55.2 mm to (74.9, 30.5)
- moved C5 53.3 mm to (39.6, 33.9), turned to 0 degrees
- moved TP5 46.2 mm to (9.65, 21.3)
- moved 3V 45.9 mm to (34.7, 37.2), turned to 270 degrees
- moved J5 44.5 mm to (34.3, 4.70)
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Routing:
- net 5V: track 162.4 -> 15.6 mm, vias 5 -> 2
- net 3V3: track 247.1 -> 137.6 mm, vias 6 -> 3
- net SDA: track 225.4 -> 170.9 mm, vias 10 -> 1
- net TX: track 17.6 -> 71.5 mm
- net RX: track 21.0 -> 73.6 mm, vias 1 -> 0
- net IMU_RESET: track 154.5 -> 103.7 mm, vias 1 -> 0
- net SA1: track 88.7 -> 39.9 mm, vias 11 -> 0
- net CS: track 52.6 -> 100.7 mm, vias 1 -> 0
- net N$17: track 43.6 -> 3.15 mm, vias 4 -> 0
- net SCL: track 213.0 -> 173.6 mm, vias 8 -> 1
- net CLK: track 58.9 -> 93.1 mm, vias 2 -> 0
- net VS: track 83.5 -> 67.1 mm, vias 7 -> 0
- net MISO: track 59.3 -> 73.7 mm, vias 1 -> 0
- net GND: track 50.8 -> 61.9 mm, vias 17 -> 3
- net N$3: track 12.5 -> 4.06 mm, vias 2 -> 0
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- added copper zone on layer 1, net 3V3
- added copper zone on layer 1, net 5V
Other:
- outline, holes or cut-outs redrawn

Commit message: remade board
Parts:
- removed TP4, TP5, TP6, TP7, TP8: TEST-POINT3, SparkFun-Connectors:PAD.03X.03
- added J1: CONN_DF13-4P-1.25DSA, X16-Pi-Shield:DF13-4P-1.25DSA
- added J2: (no value), SparkFun-Connectors:1X02
- added J6: BM04B-GHS-TBT, X16-Pi-Shield:CONN_BM04B-GHS-TBT_JST
- added U$4, U$5, U$6: TESTPOINT_5.04MM, X16-ExtraComponents:TESTPOINT_5.04MM
- moved J9 63.4 mm to (12.5, 1.36), turned to 0 degrees
- moved R12 58.5 mm to (19.9, 17.2), flipped to the bottom, turned to 180 degrees
- moved R11 57.6 mm to (19.9, 14.9), flipped to the bottom, turned to 180 degrees
- moved J5 57.5 mm to (68.7, 50.8), turned to 90 degrees
- moved J15 53.5 mm to (24.4, 1.57), turned to 180 degrees
- moved J14 53.5 mm to (30.0, 1.52), turned to 180 degrees
- moved J12 52.7 mm to (3.94, 38.6), turned to 90 degrees
- moved JP7 41.8 mm to (55.5, 21.7), turned to 0 degrees
- moved R16 38.9 mm to (36.6, 5.83), turned to 90 degrees
- moved 3V 35.3 mm to (36.6, 1.93)
- moved J11 34.9 mm to (74.7, 31.9), turned to 90 degrees
- moved C5 31.8 mm to (27.9, 4.38), flipped to the bottom, turned to 90 degrees
- moved JP5 29.2 mm to (28.7, 19.1), turned to 90 degrees
- moved JP8 28.6 mm to (27.2, 19.1), turned to 90 degrees
- moved C4 27.2 mm to (25.5, 4.41), flipped to the bottom, turned to 90 degrees
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Connections:
- new net IMU_INT_2: U$1.35, U$3.INT
- new net IMU_RESET_2: U$1.37, U$3.RST
- new net N$1: JP5.1, U1.4
- net 3V3: now also J1.1, J6.2, U$4.TP; no longer TP6.1
- net 5V: now also U$5.TP; no longer TP7.1
- net 5V_EXT: now also J2.2
- net CLK: now also J12.5; no longer J12.2
- net CS: now also J12.4; no longer J12.5
- net GND: now also J1.4, J2.1, J6.1, U$6.TP; no longer TP8.1
- net IMU_INT: no longer U$3.INT
- net IMU_RESET: no longer U$3.RST
- net MISO: now also J12.3; no longer J12.4
- net MOSI: now also J12.2; no longer J12.3
- net SA0: no longer TP4.1
- net SA1: no longer JP5.1, TP5.1, U1.4
- net SCL: now also J1.2, J6.3
- net SDA: now also J1.3, J6.4
Routing:
- net IMU_RESET: track 103.7 -> 31.4 mm
- net CS: track 100.7 -> 33.9 mm
- net GND: track 61.9 -> 5.63 mm, vias 3 -> 1
- net CLK: track 93.1 -> 41.2 mm
- net VS: track 67.1 -> 21.1 mm, vias 0 -> 3
- net 3V3: track 137.6 -> 182.4 mm, vias 3 -> 6
- net TX: track 71.5 -> 27.8 mm
- net RX: track 73.6 -> 30.0 mm
- net IMU_RESET_2: track 0.00 -> 43.5 mm
- net 5V: track 15.6 -> 59.0 mm, vias 2 -> 3
- net MISO: track 73.7 -> 42.2 mm
- net IMU_INT: track 70.9 -> 43.1 mm
- net MOSI: track 65.1 -> 37.4 mm
- net IMU_INT_2: track 0.00 -> 26.4 mm
- net SA1: track 39.9 -> 13.9 mm
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- removed copper zone on layer 1, net 3V3
- removed copper zone on layer 1, net 5V
Other:
- board size 81.3 x 74.3 mm -> 80 x 74.3 mm
