File: X16-Pi-Shield.brd (EAGLE design)
At the start: 80 x 74.3 mm, 37 parts, among them J1 CONN_DF13-4P-1.25DSA, J3 CONN_DF13-4P-1.25DSA, J4 HTST-110-04-L-D-RA, J5 BM04B-GHS-TBT, J6 BM04B-GHS-TBT, U1 INA260AIPW, U2 AZ1117IH-3.3TRG1

Commit message: finished board
Parts:
- moved 3V 38.3 mm to (20.8, 36.8), turned to 90 degrees
- moved R16 31.7 mm to (20.8, 33.3), turned to 270 degrees
- moved R15 19.3 mm to (26.6, 5.03), turned to 180 degrees
- moved 5V 13.9 mm to (32.4, 5.03), turned to 0 degrees
- moved U$5 10.4 mm to (39.8, 3.45)
- moved J11 9.18 mm to (73.5, 41.0), turned to 270 degrees
- moved U$4 8.70 mm to (49.5, 3.38)
- moved C4 8.44 mm to (23.9, 12.7), turned to 180 degrees
- moved C5 7.31 mm to (23.8, 10.5), turned to 180 degrees
- moved JP8 6.75 mm to (33.9, 18.3)
- moved JP5 5.80 mm to (34.0, 16.8), turned to 0 degrees
- moved J2 4.54 mm to (0.44, 2.91), turned to 90 degrees
- moved J7 3.73 mm to (73.4, 25.3), turned to 90 degrees
- moved U1 3.57 mm to (28.6, 17.7), turned to 180 degrees
- moved U2 3.23 mm to (31.0, 10.4), turned to 180 degrees
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Connections:
- net SCL: now also J11.3; no longer J11.2
- net SDA: now also J11.2; no longer J11.3
Routing:
- net 3V3: track 182.4 -> 223.9 mm, vias 6 -> 4
- net 5V_EXT: track 49.6 -> 71.4 mm, vias 1 -> 3
- net VS: track 21.1 -> 31.2 mm
- net ALERT: track 46.2 -> 53.2 mm
- net SDA: track 146.7 -> 153.0 mm, vias 3 -> 5
- net TX: track 27.8 -> 22.2 mm
- net GND: track 5.63 -> 0.00 mm, vias 1 -> 0
- net RX: track 30.0 -> 24.9 mm
- net SCL: track 155.7 -> 160.4 mm, vias 5 -> 7
- net IMU_INT_2: track 26.4 -> 30.6 mm
- net IMU_RESET: track 31.4 -> 27.2 mm, vias 0 -> 1
- net 5V: track 59.0 -> 62.9 mm, vias 3 -> 2
- net CLK: track 41.2 -> 44.9 mm
- net 3VO: track 29.2 -> 32.3 mm, vias 0 -> 1
- net CS: track 33.9 -> 36.1 mm
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Other:
- board text added: "3.3V"
- board text added: "5V"
- board text added: "5V Ext"
- board text added: "Alert"
- board text added: "CLK"
- board text added: "CLK CS MISO MOSI GND"
- board text added: "CS"
- board text added: "CTRL"
- board text added: "GND"
- board text added: "GND RX TX 3.3V GND 3.3V GND"
- board text added: "GND SDA SCL 3.3V"
- board text added: "GPIO"
- board text added: "IMU Int New"
- board text added: "IMU Int Old"
- board text added: "IMU Reset"
- board text added: "IMU Reset New"
- board text added: "MISO"
- board text added: "MOSI"
- board text added: "RX"
- board text added: "SA0"
- board text added: "SA1"
- board text added: "SAlert"
- board text added: "SCL"
- board text added: "SDA"
- board text added: "SDA SCL GND"
- board text added: "TX"

Commit message: board
Parts:
- moved R16 8.04 mm to (28.8, 33.3)
- moved 3V 8.01 mm to (28.8, 36.7)
Changed lines of the file:
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@@
 <text x="-0.4445" y="-0.3175" size="1.778" layer="21">GND</text>
 <text x="11.0617" y="-0.9398" size="0.762" layer="21">GND    RX     TX       3.3V     GND     3.3V     GND</text>
-<text x="72.6059" y="42.8244" size="1.27" layer="21">GND
+<text x="75.0951" y="34.3027" size="1.016" layer="21">GND
 SDA
 SCL
 3.3V</text>
-<text x="72.9615" y="18.3261" size="1.27" layer="21">SDA
+<text x="75.0316" y="25.3746" size="1.016" layer="21">SDA
 SCL
 GND</text>
@@
 </autorouter>
 <elements>
-<element name="3V" library="SparkFun-LED" package="LED-0603" value="" x="20.7899" y="36.7792" smashed="yes" rot="R90">
-<attribute name="NAME" x="20.1549" y="36.7792" size="0.6096" layer="25" font="vector" ratio="20" rot="R90" align="bottom-center"/>
-<attribute name="VALUE" x="21.4249" y="36.7792" size="0.6096" layer="27" font="vector" ratio="20" rot="R90" align="top-center"/>
+<element name="3V" library="SparkFun-LED" package="LED-0603" value="" x="28.8036" y="36.6903" smashed="yes" rot="R90">
+<attribute name="NAME" x="28.1686" y="36.6903" size="0.6096" layer="25" font="vector" ratio="20" rot="R90" align="bottom-center"/>
+<attribute name="VALUE" x="29.4386" y="36.6903" size="0.6096" layer="27" font="vector" ratio="20" rot="R90" align="top-center"/>
 </element>
 <element name="5V" library="SparkFun-LED" package="LED-0603" value="" x="32.4231" y="5.0292" smashed="yes">
@@
 <attribute name="VALUE" x="26.5811" y="5.7912" size="0.6096" layer="27" font="vector" ratio="20" rot="R180" align="top-center"/>
 </element>
-<element name="R16" library="SparkFun-Resistors" package="0603" value="60" x="20.7899" y="33.3248" smashed="yes" rot="R270">
-<attribute name="NAME" x="21.5519" y="33.3248" size="0.6096" layer="25" font="vector" ratio="20" rot="R270" align="bottom-center"/>
-<attribute name="PROD_ID" value=" " x="-141.7701" y="-35.2552" size="1.778" layer="27" rot="R270" display="off"/>
-<attribute name="VALUE" x="20.0279" y="33.3248" size="0.6096" layer="27" font="vector" ratio="20" rot="R270" align="top-center"/>
+<element name="R16" library="SparkFun-Resistors" package="0603" value="60" x="28.829" y="33.3248" smashed="yes" rot="R270">
+<attribute name="NAME" x="29.591" y="33.3248" size="0.6096" layer="25" font="vector" ratio="20" rot="R270" align="bottom-center"/>
+<attribute name="PROD_ID" value=" " x="-133.731" y="-35.2552" size="1.778" layer="27" rot="R270" display="off"/>
+<attribute name="VALUE" x="28.067" y="33.3248" size="0.6096" layer="27" font="vector" ratio="20" rot="R270" align="top-center"/>
 </element>
 <element name="U$1" library="X16-Pi-Shield" package="RPI4" value="RPI4" x="68.58" y="3.81" smashed="yes" rot="R90"/>
@@
 <wire x1="61.0997" y1="50.1777" x2="65.3034" y2="50.1777" width="0.508" layer="1"/>
 <wire x1="60.071" y1="62.9285" x2="60.5155" y2="62.484" width="0.508" layer="1"/>
-<wire x1="44.7303" y1="31.8389" x2="40.8813" y2="31.8389" width="0.508" layer="1"/>
-<wire x1="40.8432" y1="31.877" x2="40.8813" y2="31.8389" width="0.508" layer="1"/>
 <wire x1="44.7303" y1="31.8389" x2="44.7303" y2="28.7773" width="0.508" layer="1"/>
 <wire x1="44.7303" y1="28.7773" x2="44.7675" y2="28.7401" width="0.508" layer="1"/>
@@
 <wire x1="18.4531" y1="32.4866" x2="17.3482" y2="32.4866" width="0.508" layer="16"/>
 <wire x1="20.662" y1="20.7527" x2="18.9611" y2="22.4536" width="0.508" layer="16"/>
-<wire x1="17.3482" y1="32.4866" x2="20.7781" y2="32.4866" width="0.508" layer="1"/>
-<wire x1="20.7781" y1="32.4866" x2="20.7899" y2="32.4748" width="0.508" layer="1"/>
-<wire x1="40.8432" y1="31.877" x2="23.3553" y2="31.877" width="0.508" layer="1"/>
-<wire x1="22.7457" y1="32.4866" x2="20.7781" y2="32.4866" width="0.508" layer="1"/>
-<wire x1="23.3553" y1="31.877" x2="22.7457" y2="32.4866" width="0.508" layer="1"/>
+<wire x1="17.3482" y1="32.4866" x2="28.8172" y2="32.4866" width="0.508" layer="1"/>
+<wire x1="28.8172" y1="32.4866" x2="28.829" y2="32.4748" width="0.508" layer="1"/>
 <wire x1="27.4447" y1="1.524" x2="29.1846" y2="-0.2159" width="0.508" layer="1"/>
 <wire x1="29.1846" y1="-0.2159" x2="48.006" y2="-0.2159" width="0.508" layer="1"/>
 <wire x1="48.006" y1="-0.2159" x2="49.5173" y2="1.2954" width="0.508" layer="1"/>
 <wire x1="49.5173" y1="1.2954" x2="49.5173" y2="3.3782" width="0.508" layer="1"/>
+<wire x1="28.829" y1="32.4748" x2="37.7308" y2="32.4748" width="0.508" layer="1"/>
+<wire x1="37.7308" y1="32.4748" x2="38.3667" y2="31.8389" width="0.508" layer="1"/>
+<wire x1="38.3667" y1="31.8389" x2="44.7303" y2="31.8389" width="0.508" layer="1"/>
+<wire x1="44.7303" y1="31.8389" x2="40.8432" y2="31.877" width="0" layer="19" extent="1-1"/>
 </signal>
 <signal name="SCL">
@@
 <contactref element="R16" pad="1"/>
 <contactref element="3V" pad="A"/>
-<wire x1="20.7899" y1="35.9022" x2="20.7899" y2="34.1748" width="0.508" layer="1"/>
+<wire x1="28.829" y1="34.1748" x2="28.829" y2="35.7879" width="0.508" layer="1"/>
+<wire x1="28.829" y1="35.7879" x2="28.8036" y2="35.8133" width="0.508" layer="1"/>
 </signal>
 <signal name="5V_EXT">

Commit message: push
Parts:
- added 5V1: (no value), SparkFun-LED:LED-0603
- added JP1: (no value), X16-ExtraComponents:1X03
- added R1: 150, SparkFun-Resistors:0603
- moved 3V 25.6 mm to (37.4, 12.6)
- moved R16 25.6 mm to (37.5, 9.27)
- moved JP5 1.12 mm to (33.9, 15.6)
- moved JP8 0.33 mm to (33.9, 18.6)
Connections:
- removed net 3VO: U$2.3VO, U$3.3VO
- new net LEAK: JP1.1, U$1.32
- new net N$3: U$2.3VO
- new net N$5: U$3.3VO
- new net N$6: 5V1.A, R1.1
- net 3V3: now also JP1.2
- net 5V_EXT: now also R1.2
- net GND: now also 5V1.C, JP1.3
Routing:
- net 3V3: track 223.9 -> 286.3 mm
- net 3VO: track 32.3 -> 0.00 mm, vias 1 -> 0
- net LEAK: track 0.00 -> 20.9 mm
- net 5V_EXT: track 71.4 -> 76.3 mm
- net ALERT: track 53.2 -> 48.5 mm
- net N$6: track 0.00 -> 2.99 mm
- net N$1: track 2.40 -> 3.36 mm
- net VS: track 31.2 -> 31.9 mm
Other:
- board text added: "5V_EXT LED"
- board text added: "X16 Pi Shield; By Sahil Mitra; Leads: Danial, Minh, Raghav, Vijay"
