File: X16-Pi-Shield.brd (EAGLE design)
At the start: 80 x 74.3 mm, 40 parts, among them J1 CONN_DF13-4P-1.25DSA, J3 CONN_DF13-4P-1.25DSA, J4 HTST-110-04-L-D-RA, J5 BM04B-GHS-TBT, J6 BM04B-GHS-TBT, U1 INA260AIPW, U2 AZ1117IH-3.3TRG1

Commit message: Minh Update
Parts:
- C1, C2: value 120uF -> 10uF
- C4: value 10uF -> 2.2uF
- C5: value 22uF -> 2.2uF
- R1, R15: value 150 -> (none)
- R11, R12: value 10k -> (none)
- R16: value 60 -> (none)
- moved R11 0.27 mm to (20.2, 14.7)
- moved R12 0.27 mm to (20.2, 17.2)
- moved U$3 0.13 mm to (49.0, 54.0)
- renumbered 5V1 to 5V_EXT
Routing:
- net SCL: track 160.4 -> 161.1 mm
Other:
- board text added: "3V3"
- board text added: "5VEXT"
- board text added: "BNO055"
- board text added: "BNO080"
- board text added: "C:/Users/Minh/Downloads/1-victoria-royale-pegatina.bmp"
- board text added: "C:/Users/Minh/Downloads/bc13a8a0-138e-4d12-b07c-a789e0a8028b-profile_banner-480.bmp"
- board text added: "LEAK"
- board text added: "SOL1"
- board text added: "SOL2"
- board text added: "SOL3"
- board text added: "SOL4"
- board text added: "SOL5"
- board text added: "SOL6"
- board text added: "SOL7"
- board text added: "SOL8"
- board text removed: "5V Ext"
- board text removed: "5V_EXT LED"
- board text removed: "CLK CS MISO MOSI GND"
- board text removed: "GND RX TX 3.3V GND 3.3V GND"
- board text removed: "GND SDA SCL 3.3V"
- board text removed: "GPIO"
- board text removed: "SDA SCL GND"

Commit message: Minh Update 2
Parts:
- 3V, 5V, 5V_EXT: device SparkFun-LED:LED-0603 -> led:CHIPLED_0805
- moved 5V 1.23 mm to (31.2, 5.04), turned to 270 degrees
- moved 5V_EXT 0.55 mm to (0.74, 18.2), turned to 0 degrees
- moved 3V 0.35 mm to (37.5, 13.0), turned to 0 degrees
Routing:
- net N$7: track 4.11 -> 2.71 mm
- net N$6: track 2.99 -> 2.25 mm
Changed lines of the file:
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@@
 <layer number="21" name="tPlace" color="7" fill="1" visible="yes" active="yes"/>
 <layer number="22" name="bPlace" color="7" fill="1" visible="yes" active="yes"/>
-<layer number="23" name="tOrigins" color="15" fill="1" visible="no" active="yes"/>
-<layer number="24" name="bOrigins" color="15" fill="1" visible="no" active="yes"/>
+<layer number="23" name="tOrigins" color="15" fill="1" visible="yes" active="yes"/>
+<layer number="24" name="bOrigins" color="15" fill="1" visible="yes" active="yes"/>
 <layer number="25" name="tNames" color="7" fill="1" visible="yes" active="yes"/>
 <layer number="26" name="bNames" color="7" fill="1" visible="yes" active="yes"/>
@@
 </autorouter>
 <elements>
-<element name="3V" library="SparkFun-LED" library_urn="urn:adsk.eagle:library:529" package="LED-0603" package3d_urn="urn:adsk.eagle:package:39354/1" value="" x="37.4396" y="12.6365" smashed="yes" rot="R90">
-<attribute name="NAME" x="36.4236" y="12.6365" size="1.016" layer="25" font="vector" ratio="15" rot="R90" align="bottom-center"/>
-<attribute name="VALUE" x="38.0746" y="12.6365" size="0.6096" layer="27" font="vector" ratio="20" rot="R90" align="top-center"/>
-</element>
-<element name="5V" library="SparkFun-LED" library_urn="urn:adsk.eagle:library:529" package="LED-0603" package3d_urn="urn:adsk.eagle:package:39354/1" value="" x="32.4231" y="5.0292" smashed="yes">
-<attribute name="NAME" x="32.4231" y="6.0452" size="1.016" layer="25" font="vector" ratio="15" align="bottom-center"/>
-<attribute name="VALUE" x="32.4231" y="4.3942" size="0.6096" layer="27" font="vector" ratio="20" align="top-center"/>
+<element name="3V" library="led" library_urn="urn:adsk.eagle:library:259" package="CHIPLED_0805" package3d_urn="urn:adsk.eagle:package:15821/2" value="" x="37.5285" y="12.9794" smashed="yes">
+<attribute name="NAME" x="36.5506" y="13.0175" size="1.016" layer="25" font="vector" ratio="15" rot="R90" align="bottom-center"/>
+<attribute name="POPULARITY" value="52" x="37.5285" y="12.9794" size="1.778" layer="27" display="off"/>
+<attribute name="VALUE" x="37.5285" y="12.3444" size="0.6096" layer="27" font="vector" ratio="20" align="top-center"/>
+</element>
+<element name="5V" library="led" library_urn="urn:adsk.eagle:library:259" package="CHIPLED_0805" package3d_urn="urn:adsk.eagle:package:15821/2" value="" x="31.1912" y="5.0419" smashed="yes" rot="R270">
+<attribute name="NAME" x="33.9471" y="4.5212" size="1.016" layer="25" font="vector" ratio="15" align="bottom-center"/>
+<attribute name="POPULARITY" value="52" x="31.1912" y="5.0419" size="1.778" layer="27" rot="R270" display="off"/>
+<attribute name="VALUE" x="30.5562" y="5.0419" size="0.6096" layer="27" font="vector" ratio="20" rot="R270" align="top-center"/>
 </element>
 <element name="C1" library="SparkFun-Capacitors" library_urn="urn:adsk.eagle:library:510" package="0603-POLAR" package3d_urn="urn:adsk.eagle:package:37422/1" value="10uF" x="11.43" y="12.2174" smashed="yes" rot="MR180">
@@
 <attribute name="VALUE" x="-2.9718" y="58.42" size="1.27" layer="27" rot="R270"/>
 </element>
-<element name="5V_EXT" library="SparkFun-LED" library_urn="urn:adsk.eagle:library:529" package="LED-0603" package3d_urn="urn:adsk.eagle:package:39354/1" value="" x="0.6985" y="18.7706" smashed="yes" rot="R90">
-<attribute name="NAME" x="2.4765" y="18.7706" size="1.016" layer="25" font="vector" ratio="15" rot="R90" align="bottom-center"/>
-<attribute name="VALUE" x="1.3335" y="18.7706" size="0.6096" layer="27" font="vector" ratio="20" rot="R90" align="top-center"/>
+<element name="5V_EXT" library="led" library_urn="urn:adsk.eagle:library:259" package="CHIPLED_0805" package3d_urn="urn:adsk.eagle:package:15821/2" value="" x="0.7366" y="18.2245" smashed="yes">
+<attribute name="NAME" x="1.2065" y="22.5806" size="1.016" layer="25" font="vector" ratio="15" rot="R90" align="bottom-center"/>
+<attribute name="POPULARITY" value="52" x="0.7366" y="18.2245" size="1.778" layer="27" display="off"/>
+<attribute name="VALUE" x="0.7366" y="17.5895" size="0.6096" layer="27" font="vector" ratio="20" align="top-center"/>
 </element>
 <element name="R1" library="SparkFun-Resistors" library_urn="urn:adsk.eagle:library:532" package="0603" package3d_urn="urn:adsk.eagle:package:39650/1" value=" " x="0.7366" y="14.0716" smashed="yes" rot="R270">
@@
 <via x="6.35" y="5.08" extent="1-16" drill="0.35"/>
 <via x="2.54" y="8.89" extent="1-16" drill="0.35"/>
-<via x="1.27" y="21.59" extent="1-16" drill="0.35"/>
 <via x="1.27" y="25.4" extent="1-16" drill="0.35"/>
 <via x="1.27" y="29.21" extent="1-16" drill="0.35"/>
@@
 <contactref element="R15" pad="1"/>
 <contactref element="5V" pad="A"/>
-<wire x1="27.4311" y1="5.0292" x2="31.5461" y2="5.0292" width="0.508" layer="1"/>
+<wire x1="30.1412" y1="5.0419" x2="27.435165625" y2="5.033265625" width="0.508" layer="1"/>
+<wire x1="27.4311" y1="5.0292" x2="27.435165625" y2="5.033265625" width="0.508" layer="1"/>
 </signal>
 <signal name="N$9">
 <contactref element="R16" pad="1"/>
 <contactref element="3V" pad="A"/>
-<wire x1="37.465" y1="10.121" x2="37.465" y2="11.7341" width="0.508" layer="1"/>
-<wire x1="37.465" y1="11.7341" x2="37.4396" y2="11.7595" width="0.508" layer="1"/>
+<wire x1="37.5285" y1="11.9294" x2="37.465" y2="11.8659" width="0.508" layer="1"/>
+<wire x1="37.465" y1="11.8659" x2="37.465" y2="10.121" width="0.508" layer="1"/>
 </signal>
 <signal name="5V_EXT">
@@
 <contactref element="R1" pad="1"/>
 <contactref element="5V_EXT" pad="A"/>
-<wire x1="0.6985" y1="17.8936" x2="0.6985" y2="14.9597" width="0.508" layer="1"/>
-<wire x1="0.6985" y1="14.9597" x2="0.7366" y2="14.9216" width="0.508" layer="1"/>
+<wire x1="0.7366" y1="17.1745" x2="0.7366" y2="14.9216" width="0.508" layer="1"/>
 </signal>
 </signals>

Commit message: Added resistor values. Make sure to update BOM!
Parts:
- R1, R15: value (none) -> 250
- R11, R12: value (none) -> 10k
- R16: value (none) -> 150
Changed lines of the file:
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@@
 <attribute name="VALUE" x="9.7663" y="10.8077" size="0.6096" layer="27" font="vector" ratio="20" rot="R180" align="top-center"/>
 </element>
-<element name="R11" library="SparkFun-Resistors" library_urn="urn:adsk.eagle:library:532" package="0603" package3d_urn="urn:adsk.eagle:package:39650/1" value=" " x="20.193" y="14.7066" smashed="yes" rot="MR180">
+<element name="R11" library="SparkFun-Resistors" library_urn="urn:adsk.eagle:library:532" package="0603" package3d_urn="urn:adsk.eagle:package:39650/1" value="10k" x="20.193" y="14.7066" smashed="yes" rot="MR180">
 <attribute name="NAME" x="22.987" y="14.7574" size="1.016" layer="26" font="vector" ratio="15" rot="MR0" align="bottom-center"/>
 <attribute name="PROD_ID" value=" " x="77.343" y="177.2666" size="1.778" layer="28" rot="MR180" display="off"/>
 <attribute name="VALUE" x="20.193" y="15.4686" size="0.6096" layer="28" font="vector" ratio="20" rot="MR180" align="top-center"/>
 </element>
-<element name="R12" library="SparkFun-Resistors" library_urn="urn:adsk.eagle:library:532" package="0603" package3d_urn="urn:adsk.eagle:package:39650/1" value=" " x="20.1676" y="17.2085" smashed="yes" rot="MR180">
+<element name="R12" library="SparkFun-Resistors" library_urn="urn:adsk.eagle:library:532" package="0603" package3d_urn="urn:adsk.eagle:package:39650/1" value="10k" x="20.1676" y="17.2085" smashed="yes" rot="MR180">
 <attribute name="NAME" x="23.1394" y="16.7005" size="1.016" layer="26" font="vector" ratio="15" rot="MR0" align="bottom-center"/>
 <attribute name="PROD_ID" value=" " x="81.1276" y="179.7685" size="1.778" layer="28" rot="MR180" display="off"/>
 <attribute name="VALUE" x="20.1676" y="17.9705" size="0.6096" layer="28" font="vector" ratio="20" rot="MR180" align="top-center"/>
 </element>
-<element name="R15" library="SparkFun-Resistors" library_urn="urn:adsk.eagle:library:532" package="0603" package3d_urn="urn:adsk.eagle:package:39650/1" value=" " x="26.5811" y="5.0292" smashed="yes" rot="R180">
+<element name="R15" library="SparkFun-Resistors" library_urn="urn:adsk.eagle:library:532" package="0603" package3d_urn="urn:adsk.eagle:package:39650/1" value="250" x="26.5811" y="5.0292" smashed="yes" rot="R180">
 <attribute name="NAME" x="26.5049" y="6.1468" size="1.016" layer="25" font="vector" ratio="15" align="bottom-center"/>
 <attribute name="PROD_ID" value=" " x="-38.1889" y="167.5892" size="1.778" layer="27" rot="R180" display="off"/>
 <attribute name="VALUE" x="26.5811" y="5.7912" size="0.6096" layer="27" font="vector" ratio="20" rot="R180" align="top-center"/>
 </element>
-<element name="R16" library="SparkFun-Resistors" library_urn="urn:adsk.eagle:library:532" package="0603" package3d_urn="urn:adsk.eagle:package:39650/1" value=" " x="37.465" y="9.271" smashed="yes" rot="R270">
+<element name="R16" library="SparkFun-Resistors" library_urn="urn:adsk.eagle:library:532" package="0603" package3d_urn="urn:adsk.eagle:package:39650/1" value="150" x="37.465" y="9.271" smashed="yes" rot="R270">
 <attribute name="NAME" x="36.322" y="9.271" size="1.016" layer="25" font="vector" ratio="15" rot="R90" align="bottom-center"/>
 <attribute name="PROD_ID" value=" " x="-125.095" y="-59.309" size="1.778" layer="27" rot="R270" display="off"/>
@@
 <attribute name="VALUE" x="0.7366" y="17.5895" size="0.6096" layer="27" font="vector" ratio="20" align="top-center"/>
 </element>
-<element name="R1" library="SparkFun-Resistors" library_urn="urn:adsk.eagle:library:532" package="0603" package3d_urn="urn:adsk.eagle:package:39650/1" value=" " x="0.7366" y="14.0716" smashed="yes" rot="R270">
+<element name="R1" library="SparkFun-Resistors" library_urn="urn:adsk.eagle:library:532" package="0603" package3d_urn="urn:adsk.eagle:package:39650/1" value="250" x="0.7366" y="14.0716" smashed="yes" rot="R270">
 <attribute name="NAME" x="2.4384" y="14.1224" size="1.016" layer="25" font="vector" ratio="15" rot="R90" align="bottom-center"/>
 <attribute name="PROD_ID" value=" " x="-1.8288" y="13.9192" size="1.778" layer="27" rot="R270" display="off"/>

Commit message: Minh Update 3
Parts:
- R1, R15: value 250 -> (none)
- R11, R12: value 10k -> (none)
- R16: value 150 -> (none)
Changed lines of the file:
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@@
 <setting verticaltext="up"/>
 </settings>
-<grid distance="50" unitdist="mil" unit="mil" style="lines" multiple="1" display="yes" altdistance="5" altunitdist="mil" altunit="mil"/>
+<grid distance="1" unitdist="mil" unit="mil" style="lines" multiple="1" display="yes" altdistance="5" altunitdist="mil" altunit="mil"/>
 <layers>
 <layer number="1" name="Top" color="4" fill="1" visible="yes" active="yes"/>
@@
 <attribute name="VALUE" x="9.7663" y="10.8077" size="0.6096" layer="27" font="vector" ratio="20" rot="R180" align="top-center"/>
 </element>
-<element name="R11" library="SparkFun-Resistors" library_urn="urn:adsk.eagle:library:532" package="0603" package3d_urn="urn:adsk.eagle:package:39650/1" value="10k" x="20.193" y="14.7066" smashed="yes" rot="MR180">
+<element name="R11" library="SparkFun-Resistors" library_urn="urn:adsk.eagle:library:532" package="0603" package3d_urn="urn:adsk.eagle:package:39650/1" value=" " x="20.193" y="14.7066" smashed="yes" rot="MR180">
 <attribute name="NAME" x="22.987" y="14.7574" size="1.016" layer="26" font="vector" ratio="15" rot="MR0" align="bottom-center"/>
 <attribute name="PROD_ID" value=" " x="77.343" y="177.2666" size="1.778" layer="28" rot="MR180" display="off"/>
 <attribute name="VALUE" x="20.193" y="15.4686" size="0.6096" layer="28" font="vector" ratio="20" rot="MR180" align="top-center"/>
 </element>
-<element name="R12" library="SparkFun-Resistors" library_urn="urn:adsk.eagle:library:532" package="0603" package3d_urn="urn:adsk.eagle:package:39650/1" value="10k" x="20.1676" y="17.2085" smashed="yes" rot="MR180">
+<element name="R12" library="SparkFun-Resistors" library_urn="urn:adsk.eagle:library:532" package="0603" package3d_urn="urn:adsk.eagle:package:39650/1" value=" " x="20.1676" y="17.2085" smashed="yes" rot="MR180">
 <attribute name="NAME" x="23.1394" y="16.7005" size="1.016" layer="26" font="vector" ratio="15" rot="MR0" align="bottom-center"/>
 <attribute name="PROD_ID" value=" " x="81.1276" y="179.7685" size="1.778" layer="28" rot="MR180" display="off"/>
 <attribute name="VALUE" x="20.1676" y="17.9705" size="0.6096" layer="28" font="vector" ratio="20" rot="MR180" align="top-center"/>
 </element>
-<element name="R15" library="SparkFun-Resistors" library_urn="urn:adsk.eagle:library:532" package="0603" package3d_urn="urn:adsk.eagle:package:39650/1" value="250" x="26.5811" y="5.0292" smashed="yes" rot="R180">
+<element name="R15" library="SparkFun-Resistors" library_urn="urn:adsk.eagle:library:532" package="0603" package3d_urn="urn:adsk.eagle:package:39650/1" value=" " x="26.5811" y="5.0292" smashed="yes" rot="R180">
 <attribute name="NAME" x="26.5049" y="6.1468" size="1.016" layer="25" font="vector" ratio="15" align="bottom-center"/>
 <attribute name="PROD_ID" value=" " x="-38.1889" y="167.5892" size="1.778" layer="27" rot="R180" display="off"/>
 <attribute name="VALUE" x="26.5811" y="5.7912" size="0.6096" layer="27" font="vector" ratio="20" rot="R180" align="top-center"/>
 </element>
-<element name="R16" library="SparkFun-Resistors" library_urn="urn:adsk.eagle:library:532" package="0603" package3d_urn="urn:adsk.eagle:package:39650/1" value="150" x="37.465" y="9.271" smashed="yes" rot="R270">
+<element name="R16" library="SparkFun-Resistors" library_urn="urn:adsk.eagle:library:532" package="0603" package3d_urn="urn:adsk.eagle:package:39650/1" value=" " x="37.465" y="9.271" smashed="yes" rot="R270">
 <attribute name="NAME" x="36.322" y="9.271" size="1.016" layer="25" font="vector" ratio="15" rot="R90" align="bottom-center"/>
 <attribute name="PROD_ID" value=" " x="-125.095" y="-59.309" size="1.778" layer="27" rot="R270" display="off"/>
@@
 <attribute name="VALUE" x="0.7366" y="17.5895" size="0.6096" layer="27" font="vector" ratio="20" align="top-center"/>
 </element>
-<element name="R1" library="SparkFun-Resistors" library_urn="urn:adsk.eagle:library:532" package="0603" package3d_urn="urn:adsk.eagle:package:39650/1" value="250" x="0.7366" y="14.0716" smashed="yes" rot="R270">
+<element name="R1" library="SparkFun-Resistors" library_urn="urn:adsk.eagle:library:532" package="0603" package3d_urn="urn:adsk.eagle:package:39650/1" value=" " x="0.7366" y="14.0716" smashed="yes" rot="R270">
 <attribute name="NAME" x="2.4384" y="14.1224" size="1.016" layer="25" font="vector" ratio="15" rot="R90" align="bottom-center"/>
 <attribute name="PROD_ID" value=" " x="-1.8288" y="13.9192" size="1.778" layer="27" rot="R270" display="off"/>
@@
 <via x="10.16" y="1.27" extent="1-16" drill="0.35"/>
 <via x="6.35" y="1.27" extent="1-16" drill="0.35"/>
-<via x="2.54" y="1.27" extent="1-16" drill="0.35"/>
 <via x="6.35" y="5.08" extent="1-16" drill="0.35"/>
 <via x="2.54" y="8.89" extent="1-16" drill="0.35"/>
@@
 <via x="1.27" y="29.21" extent="1-16" drill="0.35"/>
 <via x="1.27" y="33.02" extent="1-16" drill="0.35"/>
-<via x="2.54" y="52.07" extent="1-16" drill="0.35"/>
 <via x="7.62" y="53.34" extent="1-16" drill="0.35"/>
 <via x="7.62" y="57.15" extent="1-16" drill="0.35"/>
@@
 <via x="1.27" y="62.23" extent="1-16" drill="0.35"/>
 <via x="4.572" y="59.69" extent="1-16" drill="0.35"/>
-<via x="11.811" y="35.179" extent="1-16" drill="0.35"/>
 </signal>
 <signal name="TX">
@@
 <wire x1="6.35" y1="22.86" x2="10.1346" y2="26.6446" width="0.254" layer="1"/>
 <wire x1="10.1346" y1="26.6446" x2="10.1346" y2="36.1696" width="0.254" layer="1"/>
-<wire x1="15.13886875" y1="36.3347" x2="16.0147" y2="37.21053125" width="0.254" layer="1"/>
-<wire x1="10.1346" y1="36.1696" x2="10.2997" y2="36.3347" width="0.254" layer="1"/>
-<wire x1="10.2997" y1="36.3347" x2="15.13886875" y2="36.3347" width="0.254" layer="1"/>
-<wire x1="16.0147" y1="37.21053125" x2="16.0147" y2="39.3954" width="0.254" layer="1"/>
+<wire x1="15.51986875" y1="36.4617" x2="16.0147" y2="36.95653125" width="0.254" layer="1"/>
+<wire x1="10.1346" y1="36.1696" x2="10.4267" y2="36.4617" width="0.254" layer="1"/>
+<wire x1="10.4267" y1="36.4617" x2="15.51986875" y2="36.4617" width="0.254" layer="1"/>
+<wire x1="16.0147" y1="36.95653125" x2="16.0147" y2="39.3954" width="0.254" layer="1"/>
 <wire x1="16.7259" y1="40.1066" x2="16.0147" y2="39.3954" width="0.254" layer="1"/>
 <wire x1="16.7259" y1="40.1066" x2="17.3482" y2="40.1066" width="0.254" layer="1"/>
@@
 <wire x1="4.0259" y1="39.8272" x2="5.0546" y2="38.7985" width="0.254" layer="16"/>
 <wire x1="11.7348" y1="38.7985" x2="11.9761" y2="38.5572" width="0.254" layer="16"/>
-<wire x1="11.9761" y1="38.5572" x2="11.9761" y2="36.5125" width="0.254" layer="16"/>
+<wire x1="11.9761" y1="38.5572" x2="11.9761" y2="36.2839" width="0.254" layer="16"/>
 <wire x1="17.3482" y1="35.2806" x2="17.3482" y2="35.0266" width="0.254" layer="16"/>
 <wire x1="5.0546" y1="38.7985" x2="11.7348" y2="38.7985" width="0.254" layer="16"/>
-<wire x1="16.3449" y1="36.2839" x2="17.3482" y2="35.2806" width="0.254" layer="16"/>
-<wire x1="11.9761" y1="36.5125" x2="12.2047" y2="36.2839" width="0.254" layer="16"/>
-<wire x1="12.2047" y1="36.2839" x2="16.3449" y2="36.2839" width="0.254" layer="16"/>
+<wire x1="16.4973" y1="36.1315" x2="17.3482" y2="35.2806" width="0.254" layer="16"/>
+<wire x1="11.9761" y1="36.2839" x2="12.1285" y2="36.1315" width="0.254" layer="16"/>
+<wire x1="12.1285" y1="36.1315" x2="16.4973" y2="36.1315" width="0.254" layer="16"/>
 </signal>
 <signal name="IMU_INT">
@@
 <contactref element="R1" pad="2"/>
 <wire x1="0.7366" y1="13.2216" x2="0.7366" y2="11.8491" width="0.508" layer="1"/>
-<wire x1="1.27" y1="11.3157" x2="2.8448" y2="11.3157" width="0.508" layer="1"/>
-<wire x1="2.8448" y1="11.3157" x2="3.81" y2="10.3505" width="0.508" layer="1"/>
-<wire x1="3.81" y1="10.3505" x2="3.81" y2="10.16" width="0.508" layer="1"/>
+<wire x1="1.27" y1="11.3157" x2="3.3528" y2="11.3157" width="0.508" layer="1"/>
+<wire x1="3.3528" y1="11.3157" x2="3.81" y2="10.8585" width="0.508" layer="1"/>
+<wire x1="3.81" y1="10.8585" x2="3.81" y2="10.16" width="0.508" layer="1"/>
 <wire x1="0.7366" y1="11.8491" x2="1.27" y2="11.3157" width="0.508" layer="1"/>
 <wire x1="9.3599" y1="9.6647" x2="9.3599" y2="8.6106" width="0.508" layer="1"/>
