File: X16-Pi-Shield.sch (EAGLE design)
At the start: 47 parts, among them J1 CONN_DF13-4P-1.25DSA, J2 CONN_DF13-4P-1.25DSA, J3 CONN_DF13-4P-1.25DSA, J4 SAMTEC-HTST-110-04-X-D-RAJ, Q2 2.5A/30V/105mΩ, Q3 220mA/50V/3.5Ω, U1 INA260AIPW, U2 AZ1117IH-3.3TRG1, Y2 ECS-80-S-4X

Commit message: final schematic
Parts:
- added JP5, JP8: JUMPER-SMT_2_NO_SILK, SparkFun-Jumpers:JUMPER-SMT_2_NO_SILK
- added TP4, TP5: TEST-POINT3, SparkFun-Connectors:TEST-POINT3
Connections:
- new net N$3: JP8.1, U1.AO
- net SA0: now also TP4.1; no longer U1.AO
- net SA1: now also JP5.1, TP5.1
- net VS: now also JP5.2, JP8.2, U2.VOUT
Changed lines of the file:
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@@
 <part name="GND18" library="SparkFun-PowerSymbols" deviceset="GND" device=""/>
 <part name="GND19" library="SparkFun-PowerSymbols" deviceset="GND" device=""/>
+<part name="TP4" library="SparkFun-Connectors" deviceset="TEST-POINT" device="3"/>
+<part name="TP5" library="SparkFun-Connectors" deviceset="TEST-POINT" device="3"/>
+<part name="JP5" library="SparkFun-Jumpers" deviceset="JUMPER-SMT_2_NO" device="_SILK"/>
+<part name="JP8" library="SparkFun-Jumpers" deviceset="JUMPER-SMT_2_NO" device="_SILK"/>
 </parts>
 <sheets>
@@
 <attribute name="VALUE" x="248.92" y="155.194" size="1.778" layer="96" rot="R180" align="top-center"/>
 </instance>
+<instance part="TP4" gate="G$1" x="48.26" y="172.72" smashed="yes">
+<attribute name="VALUE" x="45.72" y="170.18" size="1.778" layer="96" font="vector"/>
+</instance>
+<instance part="TP5" gate="G$1" x="48.26" y="165.1" smashed="yes">
+<attribute name="NAME" x="45.72" y="167.64" size="1.778" layer="95" font="vector"/>
+<attribute name="VALUE" x="45.72" y="162.56" size="1.778" layer="96" font="vector"/>
+</instance>
+<instance part="JP5" gate="G$1" x="139.7" y="154.94" smashed="yes" rot="R180">
+<attribute name="NAME" x="139.7" y="152.146" size="1.778" layer="95" font="vector" rot="R180" align="center"/>
+<attribute name="VALUE" x="139.7" y="157.734" size="1.778" layer="96" font="vector" rot="R180" align="center"/>
+</instance>
+<instance part="JP8" gate="G$1" x="139.7" y="144.78" smashed="yes" rot="R180">
+<attribute name="NAME" x="139.7" y="141.986" size="1.778" layer="95" font="vector" rot="R180" align="center"/>
+<attribute name="VALUE" x="139.7" y="147.574" size="1.778" layer="96" font="vector" rot="R180" align="center"/>
+</instance>
 </instances>
 <busses>
@@
 <wire x1="149.86" y1="154.94" x2="144.78" y2="154.94" width="0.1524" layer="91"/>
 <label x="144.78" y="154.94" size="1.778" layer="95"/>
+<pinref part="JP5" gate="G$1" pin="1"/>
+</segment>
+<segment>
+<pinref part="TP5" gate="G$1" pin="1"/>
+<wire x1="48.26" y1="165.1" x2="40.64" y2="165.1" width="0.1524" layer="91"/>
+<label x="43.18" y="165.1" size="1.778" layer="95"/>
 </segment>
 </net>
@@
 <segment>
 <pinref part="U2" gate="G$1" pin="OUTPUT"/>
-<wire x1="238.76" y1="129.54" x2="248.92" y2="129.54" width="0.1524" layer="91"/>
+<wire x1="238.76" y1="129.54" x2="241.3" y2="129.54" width="0.1524" layer="91"/>
 <label x="248.92" y="129.54" size="1.778" layer="95"/>
+<wire x1="241.3" y1="129.54" x2="248.92" y2="129.54" width="0.1524" layer="91"/>
 <wire x1="248.92" y1="129.54" x2="261.62" y2="129.54" width="0.1524" layer="91"/>
 <wire x1="248.92" y1="129.54" x2="248.92" y2="137.16" width="0.1524" layer="91"/>
 <junction x="248.92" y="129.54"/>
 <pinref part="C5" gate="G$1" pin="2"/>
+<pinref part="U2" gate="G$1" pin="VOUT"/>
+<wire x1="238.76" y1="124.46" x2="241.3" y2="124.46" width="0.1524" layer="91"/>
+<wire x1="241.3" y1="124.46" x2="241.3" y2="129.54" width="0.1524" layer="91"/>
+<junction x="241.3" y="129.54"/>
+</segment>
+<segment>
+<pinref part="JP5" gate="G$1" pin="2"/>
+<wire x1="134.62" y1="154.94" x2="127" y2="154.94" width="0.1524" layer="91"/>
+<label x="129.54" y="154.94" size="1.778" layer="95"/>
+</segment>
+<segment>
+<pinref part="JP8" gate="G$1" pin="2"/>
+<wire x1="134.62" y1="144.78" x2="127" y2="144.78" width="0.1524" layer="91"/>
+<label x="129.54" y="144.78" size="1.778" layer="95"/>
 </segment>
 </net>
 <net name="SA0" class="0">
+<segment>
+<pinref part="TP4" gate="G$1" pin="1"/>
+<wire x1="48.26" y1="172.72" x2="40.64" y2="172.72" width="0.1524" layer="91"/>
+<label x="43.18" y="172.72" size="1.778" layer="95"/>
+</segment>
+</net>
+<net name="N$3" class="0">
 <segment>
 <pinref part="U1" gate="G$1" pin="AO"/>
 <wire x1="149.86" y1="144.78" x2="144.78" y2="144.78" width="0.1524" layer="91"/>
-<label x="144.78" y="144.78" size="1.778" layer="95"/>
-</segment>
-</net>
+<pinref part="JP8" gate="G$1" pin="1"/>
+</segment>
+</net>

Commit message: update
Parts:
- removed J1, J2: CONN_DF13-4P-1.25DSA, X16-Pi-Shield:CONN_DF13-4P-1.25DSA
- added J5: BM04B-GHS-TBT, X16-Pi-Shield:BM04B-GHS-TBT
Connections:
- net 3V3: now also J5.2; no longer J1.1, J2.1
- net GND: now also J5.1; no longer J1.4, J2.4
- net SCL: now also J5.3; no longer J1.2, J2.2
- net SDA: now also J5.4; no longer J1.3, J2.3
Changed lines of the file:
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@@
 <part name="GND8" library="SparkFun-PowerSymbols" deviceset="GND" device=""/>
 <part name="GND9" library="SparkFun-PowerSymbols" deviceset="GND" device=""/>
-<part name="J1" library="X16-Pi-Shield" deviceset="CONN_DF13-4P-1.25" device="DSA"/>
-<part name="GND10" library="SparkFun-PowerSymbols" deviceset="GND" device=""/>
-<part name="J2" library="X16-Pi-Shield" deviceset="CONN_DF13-4P-1.25" device="DSA"/>
-<part name="GND11" library="SparkFun-PowerSymbols" deviceset="GND" device=""/>
 <part name="J3" library="X16-Pi-Shield" deviceset="CONN_DF13-4P-1.25" device="DSA"/>
 <part name="GND12" library="SparkFun-PowerSymbols" deviceset="GND" device=""/>
@@
 <part name="JP5" library="SparkFun-Jumpers" deviceset="JUMPER-SMT_2_NO" device="_SILK"/>
 <part name="JP8" library="SparkFun-Jumpers" deviceset="JUMPER-SMT_2_NO" device="_SILK"/>
+<part name="J5" library="X16-Pi-Shield" deviceset="BM04B-GHS-TBT" device=""/>
+<part name="GND20" library="supply1" library_urn="urn:adsk.eagle:library:371" deviceset="GND" device=""/>
 </parts>
 <sheets>
@@
 <attribute name="VALUE" x="195.58" y="170.434" size="1.778" layer="96" font="vector" rot="R180" align="top-center"/>
 </instance>
-<instance part="J1" gate="G$1" x="127" y="48.26" smashed="yes">
-<attribute name="NAME" x="125.095" y="53.34" size="1.778" layer="95"/>
-<attribute name="VALUE" x="125.095" y="39.0525" size="1.778" layer="96"/>
-</instance>
-<instance part="GND10" gate="1" x="111.76" y="40.64" smashed="yes">
-<attribute name="VALUE" x="111.76" y="37.846" size="1.778" layer="96" font="vector" rot="R180" align="top-center"/>
-</instance>
-<instance part="J2" gate="G$1" x="147.32" y="48.26" smashed="yes">
-<attribute name="NAME" x="145.415" y="53.34" size="1.778" layer="95"/>
-<attribute name="VALUE" x="145.415" y="39.0525" size="1.778" layer="96"/>
-</instance>
-<instance part="GND11" gate="1" x="132.08" y="40.64" smashed="yes">
-<attribute name="VALUE" x="132.08" y="40.386" size="1.778" layer="96" font="vector" align="top-center"/>
-</instance>
 <instance part="J3" gate="G$1" x="170.18" y="48.26" smashed="yes">
 <attribute name="NAME" x="168.275" y="53.34" size="1.778" layer="95"/>
@@
 <instance part="GND15" gate="1" x="33.02" y="127" smashed="yes">
 <attribute name="VALUE" x="33.02" y="126.746" size="1.778" layer="96" align="top-center"/>
+</instance>
+<instance part="J5" gate="A" x="60.96" y="55.88" smashed="yes">
+<attribute name="NAME" x="65.1256" y="61.1886" size="2.0828" layer="95" ratio="6" rot="SR0"/>
+</instance>
+<instance part="GND20" gate="1" x="48.26" y="50.8" smashed="yes">
+<attribute name="VALUE" x="45.72" y="48.26" size="1.778" layer="96"/>
 </instance>
 </instances>
@@
 </segment>
 <segment>
-<pinref part="J1" gate="G$1" pin="4"/>
-<wire x1="121.92" y1="43.18" x2="111.76" y2="43.18" width="0.1524" layer="91"/>
-<pinref part="GND10" gate="1" pin="GND"/>
-</segment>
-<segment>
-<pinref part="J2" gate="G$1" pin="4"/>
-<wire x1="142.24" y1="43.18" x2="132.08" y2="43.18" width="0.1524" layer="91"/>
-<pinref part="GND11" gate="1" pin="GND"/>
-</segment>
-<segment>
 <pinref part="J3" gate="G$1" pin="4"/>
 <wire x1="165.1" y1="43.18" x2="154.94" y2="43.18" width="0.1524" layer="91"/>
@@
 <label x="30.48" y="132.08" size="1.778" layer="95" rot="R270"/>
 <pinref part="GND15" gate="1" pin="GND"/>
+</segment>
+<segment>
+<pinref part="J5" gate="A" pin="1"/>
+<label x="55.88" y="55.88" size="1.778" layer="95"/>
+<wire x1="60.96" y1="55.88" x2="48.26" y2="55.88" width="0.1524" layer="91"/>
+<wire x1="48.26" y1="55.88" x2="48.26" y2="53.34" width="0.1524" layer="91"/>
+<pinref part="GND20" gate="1" pin="GND"/>
 </segment>
 </net>
@@
 </segment>
 <segment>
-<pinref part="J1" gate="G$1" pin="3"/>
-<wire x1="121.92" y1="45.72" x2="114.3" y2="45.72" width="0.1524" layer="91"/>
-<label x="116.84" y="45.72" size="1.778" layer="95"/>
-</segment>
-<segment>
 <pinref part="J3" gate="G$1" pin="3"/>
 <wire x1="165.1" y1="45.72" x2="157.48" y2="45.72" width="0.1524" layer="91"/>
@@
 </segment>
 <segment>
-<pinref part="J2" gate="G$1" pin="3"/>
-<wire x1="142.24" y1="45.72" x2="134.62" y2="45.72" width="0.1524" layer="91"/>
-<label x="137.16" y="45.72" size="1.778" layer="95"/>
-</segment>
-<segment>
 <pinref part="U$2" gate="G$1" pin="SDA"/>
 <wire x1="45.72" y1="99.06" x2="40.64" y2="99.06" width="0.1524" layer="91"/>
@@
 <label x="10.16" y="149.86" size="1.778" layer="95"/>
 </segment>
+<segment>
+<pinref part="J5" gate="A" pin="4"/>
+<wire x1="60.96" y1="48.26" x2="55.88" y2="48.26" width="0.1524" layer="91"/>
+<label x="55.88" y="48.26" size="1.778" layer="95"/>
+</segment>
 </net>
 <net name="3V3" class="0">
-<segment>
-<pinref part="J1" gate="G$1" pin="1"/>
-<wire x1="121.92" y1="50.8" x2="114.3" y2="50.8" width="0.1524" layer="91"/>
-<label x="116.84" y="50.8" size="1.778" layer="95"/>
-</segment>
-<segment>
-<pinref part="J2" gate="G$1" pin="1"/>
-<wire x1="142.24" y1="50.8" x2="134.62" y2="50.8" width="0.1524" layer="91"/>
-<label x="137.16" y="50.8" size="1.778" layer="95"/>
-</segment>
 <segment>
 <pinref part="J3" gate="G$1" pin="1"/>
@@
 <label x="33.02" y="167.64" size="1.778" layer="95" rot="R90"/>
 </segment>
+<segment>
+<pinref part="J5" gate="A" pin="2"/>
+<wire x1="60.96" y1="53.34" x2="55.88" y2="53.34" width="0.1524" layer="91"/>
+<label x="55.88" y="53.34" size="1.778" layer="95"/>
+</segment>
 </net>
 <net name="SCL" class="0">
-<segment>
-<pinref part="J1" gate="G$1" pin="2"/>
-<wire x1="121.92" y1="48.26" x2="114.3" y2="48.26" width="0.1524" layer="91"/>
-<label x="116.84" y="48.26" size="1.778" layer="95"/>
-</segment>
-<segment>
-<pinref part="J2" gate="G$1" pin="2"/>
-<wire x1="142.24" y1="48.26" x2="134.62" y2="48.26" width="0.1524" layer="91"/>
-<label x="137.16" y="48.26" size="1.778" layer="95"/>
-</segment>
 <segment>
 <pinref part="J3" gate="G$1" pin="2"/>
@@
 <label x="12.7" y="152.4" size="1.778" layer="95"/>
 </segment>
-</net>
+<segment>
+<pinref part="J5" gate="A" pin="3"/>
+<wire x1="60.96" y1="50.8" x2="55.88" y2="50.8" width="0.1524" layer="91"/>
+<label x="55.88" y="50.8" size="1.778" layer="95"/>
+</segment>
+</net>
